Commit message: update robot color

File: my_robot/urdf/my_robot.xacro (robot description, xacro)
@@ -124,5 +124,24 @@
     </visual>
     </link>
-/
+    <gazebo reference="left_wheel">
+    <material>
+      Gazebo/Orange
+    </material>
+    </gazebo>
+    <gazebo reference="right_wheel">
+    <material>
+      Gazebo/Orange
+    </material>
+    </gazebo>
+    <gazebo reference="chassis">
+    <material>
+      Gazebo/SkyBlue
+    </material>
+    </gazebo>
+    <gazebo reference="camera">
+    <material>
+      Gazebo/Yellow
+    </material>
+    </gazebo>
   <link name='chassis'>
     <pose>0 0 0.1 0 0 0</pose>
